File: STELLA RF SHIELD/EAGLE/STELLA_RF.sch (EAGLE design)
At the start: 35 parts, among them M1 WE_MCA_7488930245, Q1 ABM12W-26.0000MHZ-6-B1U-T3, U1 CC2500RGP

Commit message: add files
Other:
- note removed: "Schematic: Franz Plocksties Layout: Uwe Knüpfer"
Changed lines of the file:
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@@
 <text x="203.2" y="124.46" size="1.778" layer="95">X12</text>
 <text x="203.2" y="119.38" size="1.778" layer="95">X13</text>
-<text x="164.084" y="25.654" size="2.54" layer="106">Schematic: Franz Plocksties
-Layout: Uwe Knüpfer</text>
 <text x="251.46" y="7.62" size="2.54" layer="106">R0</text>
 <text x="174.244" y="1.27" size="2.54" layer="106">19.01.2020</text>
